File: RedPill_Rev1.2/RedPill_Rev1.2.kicad_pcb (KiCad board)
At the start: 2 copper layers, 21.6 x 66 mm, 26 parts, among them J1 Conn_01x04, J2 Conn_01x04, J3 USB_B_Mini, J5 Pin_01x20, J6 Pin_01x20, SW1 SW_Push, U1 TLV1117-33, U2 STM32G0B1KET6, X1 SG-5032CAN

Commit message: Fixed up schematic layout
Connections:
- net Net-(U1-VI) renamed /REG_VIN
- J1 pad e: GND -> (no net)
Changed lines of the file:
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@@
 			(layer "F.Mask"
 				(type "Top Solder Mask")
-				(color "Red")
+				(color "#831212FF")
 				(thickness 0.01)
 			)
@@
 			(layer "B.Mask"
 				(type "Bottom Solder Mask")
-				(color "Red")
+				(color "#831212FF")
 				(thickness 0.01)
 			)
@@
 	(net 40 "/R_LED")
 	(net 41 "/PA1")
-	(net 42 "Net-(U1-VI)")
+	(net 42 "/REG_VIN")
 	(net 43 "unconnected-(J2-Pin_2-Pad2)")
 	(footprint "LED_SMD:LED_0603_1608Metric_Pad1.05x0.95mm_HandSolder"
@@
 			(layers "F.Cu" "F.Paste" "F.Mask")
 			(roundrect_rratio 0.25)
-			(net 42 "Net-(U1-VI)")
+			(net 42 "/REG_VIN")
 			(pintype "passive")
 		)
@@
 			(layers "*.Cu" "*.Mask")
 			(remove_unused_layers no)
-			(net 1 "GND")
-			(pinfunction "Pin_4")
-			(pintype "passive")
 		)
 		(model "${KICAD8_3DMODEL_DIR}/Connector_PinHeader_2.54mm.3dshapes/PinHeader_1x04_P2.54mm_Vertical.wrl"
@@
 			(layers "F.Cu" "F.Paste" "F.Mask")
 			(roundrect_rratio 0.2)
-			(net 42 "Net-(U1-VI)")
+			(net 42 "/REG_VIN")
 			(pintype "passive")
 		)
@@
 			(layers "F.Cu" "F.Paste" "F.Mask")
 			(roundrect_rratio 0.25)
-			(net 42 "Net-(U1-VI)")
+			(net 42 "/REG_VIN")
 			(pinfunction "VI")
 			(pintype "power_in")
