File: RedPill_Rev1.2/RedPill_Rev1.2.kicad_sch (KiCad schematic)
At the start: 26 parts, among them J1 Conn_01x04, J2 Conn_01x04, J3 USB_B_Mini, J5 Pin_01x20, J6 Pin_01x20, SW1 SW_Push, U1 TLV1117-33, U2 STM32G0B1KET6, X1 SG-5032CAN

Commit message: Fixed up schematic layout
Parts:
- F1: value Polyfuse_Small -> Polyfuse
- H1: value MountingHole -> M2_2.2mm_TL
- H2: value MountingHole -> M2_2.2mm_TR
- H3: value MountingHole -> M2_2.2mm_BL
- H4: value MountingHole -> M2_2.2mm_BR
- J1, J2: value Conn_01x04 -> Pin_01x04
- SW1: value SW_Push -> PTS810
- TP5: value TestPoint -> GND Test
Connections:
- net GND: no longer J5.11 (Pin_11), J5.6 (Pin_6)
- net SYS_SWCLK: no longer J5.18 (Pin_18), U2.25 (PA14)
- net SYS_SWDIO: no longer U2.24 (PA13)
- net REG_VIN: now reaches C1.1, F1.2, U1.3 (VI)
- net REG_IN renamed DIODE_VOUT
- new net: J5.11 (Pin_11), J5.6 (Pin_6)
- new net SWCLK: J5.18 (Pin_18), U2.25 (PA14)
- new net SWDIO: U2.24 (PA13)
Other:
- note added: "CRYSTAL"
- note added: "Connects to ST-LINK V2"
- note added: "DIODE SCHOTTKY 40V 200MA 0603 SD0603S040S0R2"
- note added: "HEADER PINS"
- note added: "LED"
- note added: "LED AMBER CLEAR 0603 SMD 150060AS75000"
- note added: "MOUNTING"
- note added: "POWER MANGEMENT"
- note added: "RESET SWITCH"
- note added: "SERIAL WIRE DEBUG"
- note added: "STM32 MICROCONTROLLER"
- note added: "USB"
- note removed: "0 Ohm Jumper"
- note removed: "150060AS75000"
- note removed: "150060VS75000"
- note removed: "SD0603S040S0R2"
- company: (none) -> Miguel Valencia Robotics
- title: (none) -> RedPill STM32G0B1KET6 DevBoard
- moved on the sheet: C1, C2, C3, C4, C5, C6, D1, D2, D4, F1, H1, H2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

Commit message: v1.2a
Connections:
- net SYS_SWCLK is gone; now on net SWCLK: J1.1 (Pin_1)
- net SYS_SWDIO is gone; now on net SWDIO: J1.2 (Pin_2), J6.18 (Pin_18)
- net GND: now also J5.11 (Pin_11), J5.6 (Pin_6)
- net SHIELD: now reaches J3.6 (Shield)
- net SHIELD: now also J3.7 (Shield_2), J3.8 (Shield_3), J3.9 (Shield_4)
Other:
- moved on the sheet: J3, J5, J6, SW1, TP5
